Commit message: Fix urdf laser

File: urdf/nicla_macro.urdf.xacro (robot description, xacro)
@@ -10,5 +10,18 @@
 <xacro:property name="NICLA_IMU" value="$(arg nicla_imu)" /> <!-- TODO -->
 <xacro:macro name="nicla_box" params="name:=nicla parent_link *origin">
-    <link name="${name}_base"></link>
+    <link name="${name}_base">
+        <visual>
+            <origin xyz="0 0 0" rpy="0 0 0" />
+            <geometry>
+                <box size="0.001 0.01 0.01"/>
+            </geometry>
+        </visual>
+        <collision>
+            <origin xyz="0 0 0" rpy="0 0 0" />
+            <geometry>
+                <box size="0.001 0.01 0.01"/>
+            </geometry>
+        </collision>
+    </link>
   	<joint name="${parent_link}_to_${name}_base" type="fixed">
     	<xacro:insert_block name="origin"/>
@@ -37,5 +50,14 @@
                 <near>0.1</near>
                 <far>100</far>
-          </clip>
+            </clip>
+            <!-- <lens>
+                <intrinsics>
+                    <fx>439.597550</fx>
+                    <fy>439.597550</fy>
+                    <cx>166.12451</cx>
+                    <cy>104.41054</cy>
+                    <s>0</s>
+                </intrinsics>
+            </lens> -->
         </camera>
         <plugin name="gazebo_ros_${name}_camera_controller" filename="libgazebo_ros_camera.so">
@@ -46,14 +68,24 @@
             <cameraInfoTopicName>camera_info</cameraInfoTopicName>
             <frameName>${name}_camera</frameName>
-            <hackBaseline>0.0</hackBaseline> <!-- Set to 0.0 -->
-            <distortionK1>0.176808</distortionK1> <!-- Set to your k1 value -->
-            <distortionK2>-0.590488</distortionK2> <!-- Set to your k2 value -->
-            <distortionK3>0.0</distortionK3> <!-- Set to your k3 value -->
-            <distortionT1>-0.008412</distortionT1> <!-- Set to your p1 value -->
-            <distortionT2>0.015473</distortionT2> <!-- Set to your p2 value -->
-            <CxPrime>166.12451</CxPrime> <!-- Set to 0 -->
-            <Cx>166.12451</Cx> <!-- Set to your Cx value -->
-            <Cy>104.41054</Cy> <!-- Set to your Cy value -->
-            <focalLength>439.597550</focalLength> <!-- Set to your focal length value-->
+            <!-- Set to 0.0 -->
+            <!-- <hackBaseline>0.0</hackBaseline>  -->
+            <!-- Set to your k1 value -->
+            <!-- <distortionK1>0.176808</distortionK1>  -->
+            <!-- Set to your k2 value -->
+            <!-- <distortionK2>-0.590488</distortionK2>  -->
+            <!-- Set to your k3 value -->
+            <!-- <distortionK3>0.0</distortionK3>  -->
+            <!-- Set to your p1 value -->
+            <!-- <distortionT1>-0.008412</distortionT1>  -->
+            <!-- Set to your p2 value -->
+            <!-- <distortionT2>0.015473</distortionT2>  -->
+            <!-- Set to 0 -->
+            <!-- <CxPrime>166.12451</CxPrime>  -->
+            <!-- Set to your Cx value -->
+            <!-- <Cx>166.12451</Cx>  -->
+            <!-- Set to your Cy value -->
+            <!-- <Cy>104.41054</Cy>  -->
+            <!-- Set to your focal length value-->
+            <!-- <focalLength>439.597550</focalLength>  -->
         <!--
         Camera matrix K:
@@ -78,5 +110,5 @@
         <link name="${name}_tof"></link>
         <joint name="${name}_base_to_tof" type="fixed">
-            <origin xyz="0 0 0" rpy="0 ${-PI/2} 0"/>
+            <origin xyz="0 0 0" rpy="0 0 0"/>
             <parent link="${name}_base"/>
             <child link="${name}_tof"/>

Commit message: simulated nicla

File: urdf/nicla_macro.urdf.xacro (robot description, xacro)
@@ -4,23 +4,43 @@
 <xacro:arg name="nicla_tof" default="true"/>
 <xacro:arg name="nicla_tof_visualize" default="true"/>
-<xacro:arg name="nicla_imu" default="false"/> <!-- TODO -->
+<xacro:arg name="nicla_mic" default="true"/>
+<xacro:arg name="nicla_imu" default="true"/>
+<xacro:arg name="use_mesh" default="true"/>
 <xacro:property name="NICLA_CAMERA" value="$(arg nicla_camera)" />
 <xacro:property name="NICLA_TOF" value="$(arg nicla_tof)" />
 <xacro:property name="nicla_tof_visualize" value="$(arg nicla_tof_visualize)" />
-<xacro:property name="NICLA_IMU" value="$(arg nicla_imu)" /> <!-- TODO -->
+<xacro:property name="NICLA_MIC" value="$(arg nicla_mic)" />
+<xacro:property name="NICLA_IMU" value="$(arg nicla_imu)" />
+<xacro:property name="USE_MESH" value="$(arg use_mesh)"/>
+<xacro:property name="PI_2" value="1.57079632679" />
+<xacro:property name="PI" value="3.14159265359" />
 <xacro:macro name="nicla_box" params="name:=nicla parent_link *origin">
     <link name="${name}_base">
         <visual>
-            <origin xyz="0 0 0" rpy="0 0 0" />
-            <geometry>
-                <box size="0.001 0.01 0.01"/>
-            </geometry>
+            <xacro:if value="${USE_MESH}">
+                <origin xyz="-0.01143 -0.01143 0" rpy="0 0 0" />
+                <geometry>
+                    <mesh filename="package://nicla_vision_ros/urdf/meshes/niclavision.dae" scale="0.001 0.001 0.001" />
+                    <!-- <mesh filename="package://nicla_vision_ros/urdf/meshes/niclavision.stl" scale="0.001 0.001 0.001" /> -->
+                </geometry>
+            </xacro:if>
+            <xacro:unless value="${USE_MESH}">
+                <origin xyz="0 0 0" rpy="0 0 0" />
+                <geometry>
+                    <box size="0.02286  0.02286 0.004"/>
+                </geometry>
+            </xacro:unless>
         </visual>
         <collision>
             <origin xyz="0 0 0" rpy="0 0 0" />
             <geometry>
-                <box size="0.001 0.01 0.01"/>
+                <box size="0.02286  0.02286 0.004"/>
             </geometry>
         </collision>
+        <inertial>
+            <origin xyz="0 0 0" rpy="0 0 0" />
+            <mass value="0.01"/>
+            <inertia ixx="0.01"  ixy="0"  ixz="0" iyy="0.01" iyz="0" izz="0.01" />
+        </inertial>
     </link>
   	<joint name="${parent_link}_to_${name}_base" type="fixed">
@@ -32,5 +52,5 @@
         <link name="${name}_camera"></link>
         <joint name="${name}_base_to_camera" type="fixed">
-            <origin xyz="0 0 0" rpy="0 0 0"/>
+            <origin xyz="-0.00255 0.00778 0.0045" rpy="0 ${-PI_2} ${PI/2}"/>
             <parent link="${name}_base"/>
             <child link="${name}_camera"/>
@@ -110,5 +130,5 @@
         <link name="${name}_tof"></link>
         <joint name="${name}_base_to_tof" type="fixed">
-            <origin xyz="0 0 0" rpy="0 0 0"/>
+            <origin xyz="-0.003 0.0032 0.0017" rpy="0 ${-PI_2} 0"/>
             <parent link="${name}_base"/>
             <child link="${name}_tof"/>
@@ -119,5 +139,5 @@
         <pose>0 0 0 0 0 0</pose>
         <visualize>${nicla_tof_visualize}</visualize>
-        <update_rate>60</update_rate>
+        <update_rate>50</update_rate>
         <ray>
             <scan>
@@ -131,5 +151,5 @@
             <range>
             <min>0.04</min>
-            <max>3</max>
+            <max>4</max>
             <resolution>0.03</resolution>
             </range>
@@ -147,4 +167,40 @@
         </gazebo>
     </xacro:if>
+    <xacro:if value="${NICLA_MIC}">
+        <link name="${name}_mic"></link>
+        <joint name="${name}_base_to_mic" type="fixed">
+            <origin xyz="-0.0073 0.0048 0.0013" rpy="0 0 0"/>
+            <parent link="${name}_base"/>
+            <child link="${name}_mic"/>
+        </joint>
+    </xacro:if>
+    <xacro:if value="${NICLA_IMU}">
+        <link name="${name}_imu"></link>
+        <joint name="${name}_base_to_imu" type="fixed">
+            <origin xyz="-0.0078 -0.0046 -0.0015" rpy="0 0 0"/>
+            <parent link="${name}_base"/>
+            <child link="${name}_imu"/>
+        </joint>
+        <gazebo reference="${name}_imu">
+            <gravity>true</gravity>
+            <sensor name="${name}_imu_sensor" type="imu">
+            <always_on>true</always_on>
+            <update_rate>100</update_rate>
+            <visualize>true</visualize>
+            <topic>{name}/imu</topic>
+            <plugin filename="libgazebo_ros_imu_sensor.so" name="imu_plugin">
+                <topicName>${name}/imu</topicName>
+                <bodyName>${name}_imu</bodyName>
+                <updateRateHZ>833</updateRateHZ>
+                <gaussianNoise>0.0</gaussianNoise>
+                <xyzOffset>0 0 0</xyzOffset>
+                <rpyOffset>0 0 0</rpyOffset>
+                <frameName>${name}_imu</frameName>
+                <initialOrientationAsReference>false</initialOrientationAsReference>
+            </plugin>
+            <pose>0 0 0 0 0 0</pose>
+            </sensor>
+        </gazebo>
+    </xacro:if>
 </xacro:macro>
 </robot>

Commit message: corrected imu frame

File: urdf/nicla_macro.urdf.xacro (robot description, xacro)
@@ -178,5 +178,5 @@
         <link name="${name}_imu"></link>
         <joint name="${name}_base_to_imu" type="fixed">
-            <origin xyz="-0.0078 -0.0046 -0.0015" rpy="0 0 0"/>
+            <origin xyz="-0.0078 -0.0046 -0.0015" rpy="${PI} 0 ${PI_2}"/>
             <parent link="${name}_base"/>
             <child link="${name}_imu"/>

Commit message: corrected simulated camera

File: urdf/nicla_macro.urdf.xacro (robot description, xacro)
@@ -6,5 +6,5 @@
 <xacro:arg name="nicla_mic" default="true"/>
 <xacro:arg name="nicla_imu" default="true"/>
-<xacro:arg name="use_mesh" default="true"/>
+<xacro:arg name="nicla_use_mesh" default="true"/>
 <xacro:property name="NICLA_CAMERA" value="$(arg nicla_camera)" />
 <xacro:property name="NICLA_TOF" value="$(arg nicla_tof)" />
@@ -12,5 +12,5 @@
 <xacro:property name="NICLA_MIC" value="$(arg nicla_mic)" />
 <xacro:property name="NICLA_IMU" value="$(arg nicla_imu)" />
-<xacro:property name="USE_MESH" value="$(arg use_mesh)"/>
+<xacro:property name="USE_MESH" value="$(arg nicla_use_mesh)"/>
 <xacro:property name="PI_2" value="1.57079632679" />
 <xacro:property name="PI" value="3.14159265359" />
@@ -71,13 +71,32 @@
                 <far>100</far>
             </clip>
-            <!-- <lens>
+            <distortion>
+                <k1>0.176808</k1>
+                <k2>-0.590488</k2>
+                <k3>0.0</k3>
+                <p1>-0.008412</p1>
+                <p2>0.015473</p2>
+                <center>0.5 0.5</center>
+            </distortion>
+            <lens>
                 <intrinsics>
-                    <fx>439.597550</fx>
-                    <fy>439.597550</fy>
+                    <!-- fx = fy = width / ( 2 * tan (hfov / 2 ) ) -->
+                    <fx>416.65053</fx>
+                    <fy>419.40464</fy>
+                    <!-- cx = ( width + 1 ) / 2 -->
                     <cx>166.12451</cx>
+                    <!-- cy = ( height + 1 ) / 2 -->
                     <cy>104.41054</cy>
                     <s>0</s>
                 </intrinsics>
-            </lens> -->
+                <projection>
+                    <p_fx>421.37357</p_fx>
+                    <p_fy>426.43881</p_fy>
+                    <p_cx>160.5</p_cx>
+                    <p_cy>120.5</p_cy>
+                    <tx>0</tx>
+                    <ty>0</ty>
+                </projection>
+            </lens>
         </camera>
         <plugin name="gazebo_ros_${name}_camera_controller" filename="libgazebo_ros_camera.so">

Commit message: merging from devel - easy part

File: urdf/nicla_macro.urdf.xacro (robot description, xacro)
@@ -6,5 +6,5 @@
 <xacro:arg name="nicla_mic" default="true"/>
 <xacro:arg name="nicla_imu" default="true"/>
-<xacro:arg name="use_mesh" default="true"/>
+<xacro:arg name="nicla_use_mesh" default="true"/>
 <xacro:property name="NICLA_CAMERA" value="$(arg nicla_camera)" />
 <xacro:property name="NICLA_TOF" value="$(arg nicla_tof)" />
@@ -12,5 +12,5 @@
 <xacro:property name="NICLA_MIC" value="$(arg nicla_mic)" />
 <xacro:property name="NICLA_IMU" value="$(arg nicla_imu)" />
-<xacro:property name="USE_MESH" value="$(arg use_mesh)"/>
+<xacro:property name="USE_MESH" value="$(arg nicla_use_mesh)"/>
 <xacro:property name="PI_2" value="1.57079632679" />
 <xacro:property name="PI" value="3.14159265359" />
@@ -71,13 +71,32 @@
                 <far>100</far>
             </clip>
-            <!-- <lens>
+            <distortion>
+                <k1>0.176808</k1>
+                <k2>-0.590488</k2>
+                <k3>0.0</k3>
+                <p1>-0.008412</p1>
+                <p2>0.015473</p2>
+                <center>0.5 0.5</center>
+            </distortion>
+            <lens>
                 <intrinsics>
-                    <fx>439.597550</fx>
-                    <fy>439.597550</fy>
+                    <!-- fx = fy = width / ( 2 * tan (hfov / 2 ) ) -->
+                    <fx>416.65053</fx>
+                    <fy>419.40464</fy>
+                    <!-- cx = ( width + 1 ) / 2 -->
                     <cx>166.12451</cx>
+                    <!-- cy = ( height + 1 ) / 2 -->
                     <cy>104.41054</cy>
                     <s>0</s>
                 </intrinsics>
-            </lens> -->
+                <projection>
+                    <p_fx>421.37357</p_fx>
+                    <p_fy>426.43881</p_fy>
+                    <p_cx>160.5</p_cx>
+                    <p_cy>120.5</p_cy>
+                    <tx>0</tx>
+                    <ty>0</ty>
+                </projection>
+            </lens>
         </camera>
         <plugin name="gazebo_ros_${name}_camera_controller" filename="libgazebo_ros_camera.so">
@@ -150,7 +169,7 @@
             </scan>
             <range>
-            <min>0.04</min>
-            <max>4</max>
-            <resolution>0.03</resolution>
+                <min>0.04</min>
+                <max>3.6</max>
+                <resolution>0.03</resolution>
             </range>
             <!-- <noise>
@@ -160,7 +179,9 @@
             </noise> -->
         </ray>
-        <plugin name="gazebo_ros_${name}_tof_controller" filename="libgazebo_ros_laser.so">
+        <plugin name="gazebo_ros_${name}_tof_controller" filename="libgazebo_ros_range.so">
             <topicName>${name}/tof</topicName>
             <frameName>${name}_tof</frameName>
+            <radiation>infrared</radiation>
+            <fov>0.471239</fov>
         </plugin>
         </sensor>
@@ -178,5 +199,5 @@
         <link name="${name}_imu"></link>
         <joint name="${name}_base_to_imu" type="fixed">
-            <origin xyz="-0.0078 -0.0046 -0.0015" rpy="0 0 0"/>
+            <origin xyz="-0.0078 -0.0046 -0.0015" rpy="${PI} 0 ${PI_2}"/>
             <parent link="${name}_base"/>
             <child link="${name}_imu"/>

Commit message: camera: corrected frame for ros, added frame for gazebo, xacro args for instrinsics

File: urdf/nicla_macro.urdf.xacro (robot description, xacro)
@@ -2,4 +2,36 @@
 <robot xmlns:xacro="http://ros.org/wiki/xacro">
 <xacro:arg name="nicla_camera" default="true"/>
+<!-- ###################### CAM PARAMS ####################################
+DEFAULT CONSIDER 320x240 resolution. Distorsion should not be influenced by resolution.
+according to chagpt, for 320x320 add +40 to P_cy and K_cy
+Camera matrix K:
+                [fx, 0., cx,
+                    0., fy, cy,
+                    0., 0.,  1.] =
+[416.65053,   0.     , 166.12451,
+    0.     , 419.40464, 104.41054,
+    0.     ,   0.     ,   1.     ]
+Note:
+- ideally fx == fy
+- ideally focalLenght = fx = fy
+- focalLength = fx+fy/2 = 418.027585
+    but focalLength MUST be img_width/(2.0*(tan(HFOV/2.0))) = 439.597550
+Distortion coefficients D (OpenCV plumb_bob model):
+[k1,k2,t1,t2,k3]=[0.176808, -0.590488, -0.008412, 0.015473, 0.000000] -->
+<xacro:arg name="nicla_camera_width" default="320"/>
+<xacro:arg name="nicla_camera_height" default="240"/>
+<xacro:arg name="nicla_camera_hz" default="30.0"/>
+<!-- fx = fy = width / ( 2 * tan (hfov / 2 ) ) -->
+<xacro:arg name="nicla_camera_K_fx" default="416.65053"/>
+<xacro:arg name="nicla_camera_K_fy" default="419.40464"/>
+<!-- cx = ( width + 1 ) / 2 -->
+<xacro:arg name="nicla_camera_K_cx" default="166.12451"/>
+<!-- cy = ( height + 1 ) / 2 -->
+<xacro:arg name="nicla_camera_K_cy" default="104.41054"/>
+<xacro:arg name="nicla_camera_P_fx" default="421.373566"/>
+<xacro:arg name="nicla_camera_P_fy" default="426.438812"/>
+<xacro:arg name="nicla_camera_P_cx" default="168.731782"/>
+<xacro:arg name="nicla_camera_P_cy" default="102.665989"/>
+<!-- ###################### CAM PARAMS ########################################### -->
 <xacro:arg name="nicla_tof" default="true"/>
 <xacro:arg name="nicla_tof_visualize" default="true"/>
@@ -8,4 +40,15 @@
 <xacro:arg name="nicla_use_mesh" default="true"/>
 <xacro:property name="NICLA_CAMERA" value="$(arg nicla_camera)" />
+<xacro:property name="NICLA_CAMERA_WIDTH" value="$(arg nicla_camera_width)" />
+<xacro:property name="NICLA_CAMERA_HEIGHT" value="$(arg nicla_camera_height)" />
+<xacro:property name="NICLA_CAMERA_HZ" value="$(arg nicla_camera_hz)" />
+<xacro:property name="NICLA_CAMERA_K_fx" value="$(arg nicla_camera_K_fx)" />
+<xacro:property name="NICLA_CAMERA_K_fy" value="$(arg nicla_camera_K_fy)" />
+<xacro:property name="NICLA_CAMERA_K_cx" value="$(arg nicla_camera_K_cx)" />
+<xacro:property name="NICLA_CAMERA_K_cy" value="$(arg nicla_camera_K_cy)" />
+<xacro:property name="NICLA_CAMERA_P_fx" value="$(arg nicla_camera_P_fx)" />
+<xacro:property name="NICLA_CAMERA_P_fy" value="$(arg nicla_camera_P_fy)" />
+<xacro:property name="NICLA_CAMERA_P_cx" value="$(arg nicla_camera_P_cx)" />
+<xacro:property name="NICLA_CAMERA_P_cy" value="$(arg nicla_camera_P_cy)" />
 <xacro:property name="NICLA_TOF" value="$(arg nicla_tof)" />
 <xacro:property name="nicla_tof_visualize" value="$(arg nicla_tof_visualize)" />
@@ -52,17 +95,24 @@
         <link name="${name}_camera"></link>
         <joint name="${name}_base_to_camera" type="fixed">
-            <origin xyz="-0.00255 0.00778 0.0045" rpy="0 ${-PI_2} ${PI/2}"/>
+            <origin xyz="-0.00255 0.00778 0.0045" rpy="0 0 ${PI}"/>
             <parent link="${name}_base"/>
             <child link="${name}_camera"/>
         </joint>
+        <link name="${name}_camera_gz"></link>
+        <joint name="${name}_camera_to_camera_gz" type="fixed">
+            <!-- gazebo sensor wants the x axis forward, z up -->
+            <origin xyz="-0.00255 0.00778 0.0045" rpy="0 ${-PI_2} ${-PI/2}"/>
+            <parent link="${name}_base"/>
+            <child link="${name}_camera_gz"/>
+        </joint>
         <!-- gazebo simulated camera -->
-        <gazebo reference="${name}_camera">
-        <sensor type="camera" name="${name}_camera">
-        <update_rate>30.0</update_rate>
-        <camera name="${name}_camera">
+        <gazebo reference="${name}_camera_gz">
+        <sensor type="camera" name="${name}_camera_gz">
+        <update_rate>${NICLA_CAMERA_HZ}</update_rate>
+        <camera name="${name}_camera_gz">
             <horizontal_fov>0.69813</horizontal_fov>  <!-- 80deg 1.39626rad-->
             <image>
-                <width>320</width>
-                <height>240</height>
+                <width>${NICLA_CAMERA_WIDTH}</width>
+                <height>${NICLA_CAMERA_HEIGHT}</height>
                 <format>R8G8B8</format>
             </image>
@@ -80,30 +130,32 @@
             </distortion>
             <lens>
-                <intrinsics>
-                    <!-- fx = fy = width / ( 2 * tan (hfov / 2 ) ) -->
-                    <fx>416.65053</fx>
-                    <fy>419.40464</fy>
-                    <!-- cx = ( width + 1 ) / 2 -->
-                    <cx>166.12451</cx>
-                    <!-- cy = ( height + 1 ) / 2 -->
-                    <cy>104.41054</cy>
-                    <s>0</s>
-                </intrinsics>
                 <projection>
-                    <p_fx>421.37357</p_fx>
-                    <p_fy>426.43881</p_fy>
-                    <p_cx>160.5</p_cx>
-                    <p_cy>120.5</p_cy>
+                    <p_fx>${NICLA_CAMERA_P_fx}</p_fx>
+                    <p_fy>${NICLA_CAMERA_P_fy}</p_fy>
+                    <p_cx>${NICLA_CAMERA_P_cx}</p_cx>
+                    <p_cy>${NICLA_CAMERA_P_cy}</p_cy>
                     <tx>0</tx>
                     <ty>0</ty>
                 </projection>
+                <intrinsics>
+                    <!-- fx = fy = width / ( 2 * tan (hfov / 2 ) ) -->
+                    <fx>${NICLA_CAMERA_K_fx}</fx>
+                    <fy>${NICLA_CAMERA_K_fy}</fy>
+                    <!-- cx = ( width + 1 ) / 2 -->
+                    <cx>${NICLA_CAMERA_K_cx}</cx>
+                    <!-- cy = ( height + 1 ) / 2 -->
+                    <cy>${NICLA_CAMERA_K_cy}</cy>
+                    <s>0</s>
+                </intrinsics>
             </lens>
         </camera>
         <plugin name="gazebo_ros_${name}_camera_controller" filename="libgazebo_ros_camera.so">
             <alwaysOn>true</alwaysOn>
-            <updateRate>0.0</updateRate>
+            <updateRate>${NICLA_CAMERA_HZ}</updateRate>
             <cameraName>${name}/camera</cameraName>
             <imageTopicName>image_raw</imageTopicName>
             <cameraInfoTopicName>camera_info</cameraInfoTopicName>
+            <!-- Cam Info and camera image MUST use the ros convention (z forward, x right), so
+            frame here is ${name}_camera (i.e. the "optical") and NOT ${name}_camera_gz -->
             <frameName>${name}_camera</frameName>
             <!-- Set to 0.0 -->
@@ -127,19 +179,4 @@
             <!-- Set to your focal length value-->
             <!-- <focalLength>439.597550</focalLength>  -->
-        <!--
-        Camera matrix K:
-                        [fx, 0., cx,
-                         0., fy, cy,
-                         0., 0.,  1.] =
-        [416.65053,   0.     , 166.12451,
-           0.     , 419.40464, 104.41054,
-           0.     ,   0.     ,   1.     ]
-        Note:
-        - ideally fx == fy
-        - ideally focalLenght = fx = fy
-        - focalLength = fx+fy/2 = 418.027585
-            but focalLength MUST be img_width/(2.0*(tan(HFOV/2.0))) = 439.597550
-        Distortion coefficients D (OpenCV plumb_bob model):
-        [k1,k2,t1,t2,k3]=[0.176808, -0.590488, -0.008412, 0.015473, 0.000000] -->
         </plugin>
         </sensor>
